File: ESP32Module.sch (KiCad schematic (older format))
At the start: 27 parts, among them J8 USB_C_Receptacle, Q1 MBT3904DW1, SW1 SW_SPST, SW2 SW_SPST, U3 ESP32-WROOM-32, U4 CP2102N-A01-GQFN24

Commit message: added cm4
Parts:
- removed U4: CP2102N-A01-GQFN24, Package_DFN_QFN:QFN-24-1EP_4x4mm_P0.5mm_EP2.6x2.6mm, symbol Interface_USB:CP2102N-A01-GQFN24
- added U4: CP2102N-A01-GQFN28, Package_DFN_QFN:QFN-28-1EP_5x5mm_P0.5mm_EP3.35x3.35mm, symbol Interface_USB:CP2102N-A01-GQFN28
Connections:
- wire segments 35 -> 32
- no-connect marks 27 -> 16
Other:
- moved on the sheet: C19, C20, C21
Changed lines of the file:
@@
 Text HLabel 2050 1700 0    50   Input ~ 0
 IO39
-NoConn ~ 8000 3450
-NoConn ~ 8000 3350
-NoConn ~ 8000 3250
-NoConn ~ 8000 3150
-NoConn ~ 8000 2350
-NoConn ~ 8000 2950
-NoConn ~ 8000 2250
-Text Label 8000 2450 0    50   ~ 0
+Text Label 7250 1850 0    50   ~ 0
 RTS
-Text Label 8000 2650 0    50   ~ 0
+Text Label 7250 2050 0    50   ~ 0
 RXD
-Text Label 8100 2550 0    50   ~ 0
+Text Label 7350 1950 0    50   ~ 0
 TXD
-Text Label 8000 2850 0    50   ~ 0
+Text Label 7250 2250 0    50   ~ 0
 DTR
 Wire Wire Line
-	8000 2550 8100 2550
-NoConn ~ 8000 2750
-Wire Wire Line
-	7450 3750 7400 3750
-Wire Wire Line
-	7450 3750 7450 3850
-Connection ~ 7450 3750
-Wire Wire Line
-	7500 3750 7450 3750
-$Comp
-L power:GND #PWR0158
-U 1 1 5DAFA538
-P 7450 3850
-AR Path="/5DAA9390/5DAAB924/5DAFA538" Ref="#PWR0158"  Part="1"
-AR Path="/5DAA9E7A/5DB7E2D8/5DAFA538" Ref="#PWR?"  Part="1"
-AR Path="/5DB7E2D8/5DAFA538" Ref="#PWR?"  Part="1"
-AR Path="/5FFBF360/5DAFA538" Ref="#PWR?"  Part="1"
-AR Path="/5DAAB924/5DAFA538" Ref="#PWR077"  Part="1"
-F 0 "#PWR0158" H 7450 3600 50  0001 C CNN
-F 1 "GND" H 7455 3677 50  0000 C CNN
-F 2 "" H 7450 3850 50  0001 C CNN
-F 3 "" H 7450 3850 50  0001 C CNN
-	1    7450 3850
-	1    0    0    -1
-$EndComp
-NoConn ~ 6800 2250
-NoConn ~ 6800 2550
-Text Label 6800 3250 2    50   ~ 0
+	7250 1950 7350 1950
+Text Label 6250 2250 2    50   ~ 0
 USBD_P
-Text Label 6800 3350 2    50   ~ 0
+Text Label 6250 2350 2    50   ~ 0
 USBD_N
 Wire Wire Line
-	6800 3150 6450 3150
+	6250 2150 5900 2150
 $Comp
 L power:+3.3V #PWR0157
 U 1 1 5DDDAE64
-P 6450 3150
+P 5900 2150
 AR Path="/5DAA9390/5DAAB924/5DDDAE64" Ref="#PWR0157"  Part="1"
 AR Path="/5DAA9E7A/5DB7E2D8/5DDDAE64" Ref="#PWR?"  Part="1"
 AR Path="/5FFBF360/5DDDAE64" Ref="#PWR?"  Part="1"
 AR Path="/5DAAB924/5DDDAE64" Ref="#PWR074"  Part="1"
-F 0 "#PWR0157" H 6450 3000 50  0001 C CNN
-F 1 "+3.3V" V 6465 3278 50  0000 L CNN
-F 2 "" H 6450 3150 50  0001 C CNN
-F 3 "" H 6450 3150 50  0001 C CNN
-	1    6450 3150
+F 0 "#PWR0157" H 5900 2000 50  0001 C CNN
+F 1 "+3.3V" V 5915 2278 50  0000 L CNN
+F 2 "" H 5900 2150 50  0001 C CNN
+F 3 "" H 5900 2150 50  0001 C CNN
+	1    5900 2150
 	0    -1   -1   0
 $EndComp
@@
 L Device:C C20
 U 1 1 5DAECE2A
-P 6200 3000
+P 5650 2100
 AR Path="/5DAA9390/5DAAB924/5DAECE2A" Ref="C20"  Part="1"
 AR Path="/5DAA9E7A/5DB7E2D8/5DAECE2A" Ref="C?"  Part="1"
@@
 AR Path="/5FFBF360/5DAECE2A" Ref="C?"  Part="1"
 AR Path="/5DAAB924/5DAECE2A" Ref="C20"  Part="1"
-F 0 "C20" H 6315 3046 50  0000 L CNN
-F 1 "0.1uF" H 6315 2955 50  0000 L CNN
-F 2 "Capacitor_SMD:C_0402_1005Metric" H 6238 2850 50  0001 C CNN
-F 3 "~" H 6200 3000 50  0001 C CNN
-	1    6200 3000
+F 0 "C20" H 5765 2146 50  0000 L CNN
+F 1 "0.1uF" H 5765 2055 50  0000 L CNN
+F 2 "Capacitor_SMD:C_0402_1005Metric" H 5688 1950 50  0001 C CNN
+F 3 "~" H 5650 2100 50  0001 C CNN
+	1    5650 2100
 	1    0    0    -1
 $EndComp
@@
 L Device:C C19
 U 1 1 5DAED8B3
-P 5750 3000
+P 5200 2100
 AR Path="/5DAA9390/5DAAB924/5DAED8B3" Ref="C19"  Part="1"
 AR Path="/5DAA9E7A/5DB7E2D8/5DAED8B3" Ref="C?"  Part="1"
@@
 AR Path="/5FFBF360/5DAED8B3" Ref="C?"  Part="1"
 AR Path="/5DAAB924/5DAED8B3" Ref="C19"  Part="1"
-F 0 "C19" H 5865 3046 50  0000 L CNN
-F 1 "4.7uF" H 5865 2955 50  0000 L CNN
-F 2 "Capacitor_SMD:C_0402_1005Metric" H 5788 2850 50  0001 C CNN
-F 3 "~" H 5750 3000 50  0001 C CNN
-	1    5750 3000
-	1    0    0    -1
-$EndComp
-Wire Wire Line
-	5750 2850 6000 2850
-Connection ~ 6200 2850
-Wire Wire Line
-	6200 2850 6800 2850
-Wire Wire Line
-	5750 3150 6000 3150
+F 0 "C19" H 5315 2146 50  0000 L CNN
+F 1 "4.7uF" H 5315 2055 50  0000 L CNN
+F 2 "Capacitor_SMD:C_0402_1005Metric" H 5238 1950 50  0001 C CNN
+F 3 "~" H 5200 2100 50  0001 C CNN
+	1    5200 2100
+	1    0    0    -1
+$EndComp
+Wire Wire Line
+	5200 1950 5450 1950
+Connection ~ 5650 1950
+Wire Wire Line
+	5650 1950 6250 1950
+Wire Wire Line
+	5200 2250 5450 2250
 $Comp
 L power:GND #PWR0156
 U 1 1 5DAEE3C7
-P 6000 3150
+P 5450 2250
 AR Path="/5DAA9390/5DAAB924/5DAEE3C7" Ref="#PWR0156"  Part="1"
 AR Path="/5DAA9E7A/5DB7E2D8/5DAEE3C7" Ref="#PWR?"  Part="1"
@@
 AR Path="/5FFBF360/5DAEE3C7" Ref="#PWR?"  Part="1"
 AR Path="/5DAAB924/5DAEE3C7" Ref="#PWR073"  Part="1"
-F 0 "#PWR0156" H 6000 2900 50  0001 C CNN
-F 1 "GND" H 6005 2977 50  0000 C CNN
-F 2 "" H 6000 3150 50  0001 C CNN
-F 3 "" H 6000 3150 50  0001 C CNN
-	1    6000 3150
-	1    0    0    -1
-$EndComp
-Connection ~ 6000 3150
-Wire Wire Line
-	6000 3150 6200 3150
+F 0 "#PWR0156" H 5450 2000 50  0001 C CNN
+F 1 "GND" H 5455 2077 50  0000 C CNN
+F 2 "" H 5450 2250 50  0001 C CNN
+F 3 "" H 5450 2250 50  0001 C CNN
+	1    5450 2250
+	1    0    0    -1
+$EndComp
+Connection ~ 5450 2250
+Wire Wire Line
+	5450 2250 5650 2250
 $Comp
 L power:+3.3V #PWR0155
 U 1 1 5DAEE89E
-P 6000 2850
+P 5450 1950
 AR Path="/5DAA9390/5DAAB924/5DAEE89E" Ref="#PWR0155"  Part="1"
 AR Path="/5DAA9E7A/5DB7E2D8/5DAEE89E" Ref="#PWR?"  Part="1"
@@
 AR Path="/5FFBF360/5DAEE89E" Ref="#PWR?"  Part="1"
 AR Path="/5DAAB924/5DAEE89E" Ref="#PWR072"  Part="1"
-F 0 "#PWR0155" H 6000 2700 50  0001 C CNN
-F 1 "+3.3V" H 6015 3023 50  0000 C CNN
-F 2 "" H 6000 2850 50  0001 C CNN
-F 3 "" H 6000 2850 50  0001 C CNN
-	1    6000 2850
-	1    0    0    -1
-$EndComp
-Connection ~ 6000 2850
-Wire Wire Line
-	6000 2850 6200 2850
-NoConn ~ 6800 2650
+F 0 "#PWR0155" H 5450 1800 50  0001 C CNN
+F 1 "+3.3V" H 5465 2123 50  0000 C CNN
+F 2 "" H 5450 1950 50  0001 C CNN
+F 3 "" H 5450 1950 50  0001 C CNN
+	1    5450 1950
+	1    0    0    -1
+$EndComp
+Connection ~ 5450 1950
+Wire Wire Line
+	5450 1950 5650 1950
 $Comp
 L power:+3.3V #PWR0154
 U 1 1 5DB16B52
-P 7350 1700
+P 6700 1300
 AR Path="/5DAA9390/5DAAB924/5DB16B52" Ref="#PWR0154"  Part="1"
 AR Path="/5DAA9E7A/5DB7E2D8/5DB16B52" Ref="#PWR?"  Part="1"
@@
 AR Path="/5FFBF360/5DB16B52" Ref="#PWR?"  Part="1"
 AR Path="/5DAAB924/5DB16B52" Ref="#PWR076"  Part="1"
-F 0 "#PWR0154" H 7350 1550 50  0001 C CNN
-F 1 "+3.3V" H 7365 1873 50  0000 C CNN
-F 2 "" H 7350 1700 50  0001 C CNN
-F 3 "" H 7350 1700 50  0001 C CNN
-	1    7350 1700
+F 0 "#PWR0154" H 6700 1150 50  0001 C CNN
+F 1 "+3.3V" H 6715 1473 50  0000 C CNN
+F 2 "" H 6700 1300 50  0001 C CNN
+F 3 "" H 6700 1300 50  0001 C CNN
+	1    6700 1300
 	1    0    0    -1
 $EndComp
@@
 L Device:C C21
 U 1 1 5DB17CCD
-P 7500 1800
+P 6850 1400
 AR Path="/5DAA9390/5DAAB924/5DB17CCD" Ref="C21"  Part="1"
 AR Path="/5DAA9E7A/5DB7E2D8/5DB17CCD" Ref="C?"  Part="1"
@@
 AR Path="/5FFBF360/5DB17CCD" Ref="C?"  Part="1"
 AR Path="/5DAAB924/5DB17CCD" Ref="C21"  Part="1"
-F 0 "C21" V 7248 1800 50  0000 C CNN
-F 1 "0.1uF" V 7339 1800 50  0000 C CNN
-F 2 "Capacitor_SMD:C_0402_1005Metric" H 7538 1650 50  0001 C CNN
-F 3 "~" H 7500 1800 50  0001 C CNN
-	1    7500 1800
+F 0 "C21" V 6598 1400 50  0000 C CNN
+F 1 "0.1uF" V 6689 1400 50  0000 C CNN
+F 2 "Capacitor_SMD:C_0402_1005Metric" H 6888 1250 50  0001 C CNN
+F 3 "~" H 6850 1400 50  0001 C CNN
+	1    6850 1400
 	0    1    1    0
 $EndComp
 Wire Wire Line
-	7350 1700 7350 1800
-Connection ~ 7350 1800
-Wire Wire Line
-	7350 1800 7350 1950
+	6700 1300 6700 1400
+Connection ~ 6700 1400
+Wire Wire Line
+	6700 1400 6700 1550
 $Comp
 L power:GND #PWR0153
 U 1 1 5DB18C85
-P 7650 1800
+P 7000 1400
 AR Path="/5DAA9390/5DAAB924/5DB18C85" Ref="#PWR0153"  Part="1"
 AR Path="/5DAA9E7A/5DB7E2D8/5DB18C85" Ref="#PWR?"  Part="1"
@@
 AR Path="/5FFBF360/5DB18C85" Ref="#PWR?"  Part="1"
 AR Path="/5DAAB924/5DB18C85" Ref="#PWR079"  Part="1"
-F 0 "#PWR0153" H 7650 1550 50  0001 C CNN
-F 1 "GND" V 7655 1672 50  0000 R CNN
-F 2 "" H 7650 1800 50  0001 C CNN
-F 3 "" H 7650 1800 50  0001 C CNN
-	1    7650 1800
+F 0 "#PWR0153" H 7000 1150 50  0001 C CNN
+F 1 "GND" V 7005 1272 50  0000 R CNN
+F 2 "" H 7000 1400 50  0001 C CNN
+F 3 "" H 7000 1400 50  0001 C CNN
+	1    7000 1400
 	0    -1   -1   0
 $EndComp
 Wire Wire Line
-	7400 1950 7350 1950
-Wire Wire Line
-	7350 1950 7300 1950
-Connection ~ 7350 1950
-$Comp
-L Interface_USB:CP2102N-A01-GQFN24 U4
-U 1 1 5DA9E645
-P 7400 2850
-AR Path="/5DAA9390/5DAAB924/5DA9E645" Ref="U4"  Part="1"
-AR Path="/5DAA9E7A/5DB7E2D8/5DA9E645" Ref="U?"  Part="1"
-AR Path="/5DB7E2D8/5DA9E645" Ref="U?"  Part="1"
-AR Path="/5FFBF360/5DA9E645" Ref="U?"  Part="1"
-AR Path="/5DAAB924/5DA9E645" Ref="U4"  Part="1"
-F 0 "U4" H 7100 3650 50  0000 C CNN
-F 1 "CP2102N-A01-GQFN24" H 7900 3650 50  0000 C CNN
-F 2 "Package_DFN_QFN:QFN-24-1EP_4x4mm_P0.5mm_EP2.6x2.6mm" H 7850 2050 50  0001 L CNN
-F 3 "https://www.silabs.com/documents/public/data-sheets/cp2102n-datasheet.pdf" H 7450 1800 50  0001 C CNN
-	1    7400 2850
-	1    0    0    -1
-$EndComp
+	6750 1550 6700 1550
+Wire Wire Line
+	6700 1550 6650 1550
+Connection ~ 6700 1550
 Text Label 10000 950  3    50   ~ 0
 RTS
@@
 Text Label 10000 1400 3    50   ~ 0
 IO0
+$Comp
+L Interface_USB:CP2102N-A01-GQFN28 U4
+U 1 1 60DC4198
+P 6750 2850
+F 0 "U4" H 6750 1461 50  0000 C CNN
+F 1 "CP2102N-A01-GQFN28" H 6750 1370 50  0000 C CNN
+F 2 "Package_DFN_QFN:QFN-28-1EP_5x5mm_P0.5mm_EP3.35x3.35mm" H 7200 1650 50  0001 L CNN
+F 3 "https://www.silabs.com/documents/public/data-sheets/cp2102n-datasheet.pdf" H 6800 2100 50  0001 C CNN
+	1    6750 2850
+	1    0    0    -1
+$EndComp
+$Comp
+L power:GND #PWR0158
+U 1 1 60E0A619
+P 6750 4150
+F 0 "#PWR0158" H 6750 3900 50  0001 C CNN
+F 1 "GND" H 6755 3977 50  0000 C CNN
+F 2 "" H 6750 4150 50  0001 C CNN
+F 3 "" H 6750 4150 50  0001 C CNN
+	1    6750 4150
+	1    0    0    -1
+$EndComp
 $EndSCHEMATC
